File: PCB/power_supply.sch (KiCad schematic (older format))
At the start: 22 parts

Commit message: Nearly finished schematic
Parts:
- BT1: renamed from BT?; footprint plenoptoscope:Keystone_18650_Battery_Clip -> power_supplies:Keystone_18650_Battery_Clip
- gave numbers to parts that had none: 21

Commit message: change footprints. Add dip switch for null modem
Parts:
- removed U4: TPS73733, Package_TO_SOT_SMD:SOT-223-6_TabPin3, symbol power_supplies:TPS737xx-plenoptoscope
- added U4: AMS1117, Package_TO_SOT_SMD:SOT-223-3_TabPin2, symbol Regulator_Linear:AMS1117
- BT1: footprint power_supplies:Keystone_18650_Battery_Clip -> Connector_JST:JST_PH_B2B-PH-K_1x02_P2.00mm_Vertical
- D1, D2: footprint LED_THT:LED_D5.0mm -> LED_SMD:LED_0805_2012Metric
Connections:
- wire segments 61 -> 58
Other:
- moved on the sheet: C10, C11
Changed lines of the file:
@@
 $EndComp
 Wire Wire Line
-	9550 2900 9700 2900
-Wire Wire Line
-	9550 3200 9550 3350
-Wire Wire Line
-	9550 2900 9550 3000
-$Comp
-L power_supplies:TPS737xx-plenoptoscope U4
-U 1 1 5C7F78F3
-P 8750 3050
-F 0 "U4" H 8750 3465 50  0000 C CNN
-F 1 "TPS73733" H 8750 3374 50  0000 C CNN
-F 2 "Package_TO_SOT_SMD:SOT-223-6_TabPin3" H 8600 3350 50  0001 C CNN
-F 3 "http://www.ti.com/lit/ds/symlink/tps737.pdf" H 8600 3350 50  0001 C CNN
-F 4 "https://au.element14.com/texas-instruments/tps73733dcq/ic-voltage-regulator/dp/1703384" H 8750 3050 50  0001 C CNN "Supplier"
-F 5 "$2.64" H 8750 3050 50  0001 C CNN "Price"
-	1    8750 3050
-	1    0    0    -1
-$EndComp
-Wire Wire Line
-	7950 2900 8300 2900
-Wire Wire Line
-	8300 2900 8350 2900
+	9100 3200 9100 3250
+Wire Wire Line
+	9100 2900 9100 3000
 Connection ~ 7950 2900
 Wire Wire Line
 	7950 2900 7950 3050
-Wire Wire Line
-	9150 2900 9550 2900
-Connection ~ 9550 2900
-Wire Wire Line
-	8350 3200 8300 3200
-Wire Wire Line
-	8300 3200 8300 2900
-Connection ~ 8300 2900
 $Comp
 L power:GND #PWR027
 U 1 1 5C832AA9
-P 9550 3350
-F 0 "#PWR027" H 9550 3100 50  0001 C CNN
-F 1 "GND" H 9555 3177 50  0000 C CNN
-F 2 "" H 9550 3350 50  0001 C CNN
-F 3 "" H 9550 3350 50  0001 C CNN
-	1    9550 3350
+P 9100 3250
+F 0 "#PWR027" H 9100 3000 50  0001 C CNN
+F 1 "GND" H 9105 3077 50  0000 C CNN
+F 2 "" H 9100 3250 50  0001 C CNN
+F 3 "" H 9100 3250 50  0001 C CNN
+	1    9100 3250
 	1    0    0    -1
 $EndComp
@@
 L power:GND #PWR025
 U 1 1 5C832B16
-P 8700 3550
-F 0 "#PWR025" H 8700 3300 50  0001 C CNN
-F 1 "GND" H 8705 3377 50  0000 C CNN
-F 2 "" H 8700 3550 50  0001 C CNN
-F 3 "" H 8700 3550 50  0001 C CNN
-	1    8700 3550
+P 8750 3250
+F 0 "#PWR025" H 8750 3000 50  0001 C CNN
+F 1 "GND" H 8755 3077 50  0000 C CNN
+F 2 "" H 8750 3250 50  0001 C CNN
+F 3 "" H 8750 3250 50  0001 C CNN
+	1    8750 3250
 	1    0    0    -1
 $EndComp
@@
 $EndComp
 Wire Wire Line
-	8700 3500 8700 3550
+	8750 3200 8750 3250
 $Comp
 L Device:C_Small C9
@@
 L Device:C_Small C11
 U 1 1 5C841CF1
-P 9550 3100
-F 0 "C11" H 9642 3146 50  0000 L CNN
-F 1 "1u" H 9642 3055 50  0000 L CNN
-F 2 "Capacitor_SMD:C_0805_2012Metric" H 9550 3100 50  0001 C CNN
-F 3 "~" H 9550 3100 50  0001 C CNN
-	1    9550 3100
+P 9100 3100
+F 0 "C11" H 9192 3146 50  0000 L CNN
+F 1 "1u" H 9192 3055 50  0000 L CNN
+F 2 "Capacitor_SMD:C_0805_2012Metric" H 9100 3100 50  0001 C CNN
+F 3 "~" H 9100 3100 50  0001 C CNN
+	1    9100 3100
 	1    0    0    -1
 $EndComp
@@
 L Device:C_Small C10
 U 1 1 5C4A11C5
-P 9250 3400
-F 0 "C10" H 9342 3446 50  0000 L CNN
-F 1 "10n" H 9342 3355 50  0000 L CNN
-F 2 "Capacitor_SMD:C_0805_2012Metric" H 9250 3400 50  0001 C CNN
-F 3 "~" H 9250 3400 50  0001 C CNN
-	1    9250 3400
+P 9400 3100
+F 0 "C10" H 9492 3146 50  0000 L CNN
+F 1 "10n" H 9492 3055 50  0000 L CNN
+F 2 "Capacitor_SMD:C_0805_2012Metric" H 9400 3100 50  0001 C CNN
+F 3 "~" H 9400 3100 50  0001 C CNN
+	1    9400 3100
 	1    0    0    -1
 $EndComp
@@
 L power:GND #PWR026
 U 1 1 5C4A145F
-P 9250 3550
-F 0 "#PWR026" H 9250 3300 50  0001 C CNN
-F 1 "GND" H 9255 3377 50  0000 C CNN
-F 2 "" H 9250 3550 50  0001 C CNN
-F 3 "" H 9250 3550 50  0001 C CNN
-	1    9250 3550
-	1    0    0    -1
-$EndComp
-Wire Wire Line
-	9250 3550 9250 3500
-Wire Wire Line
-	9250 3300 9250 3200
-Wire Wire Line
-	9250 3200 9150 3200
+P 9400 3250
+F 0 "#PWR026" H 9400 3000 50  0001 C CNN
+F 1 "GND" H 9405 3077 50  0000 C CNN
+F 2 "" H 9400 3250 50  0001 C CNN
+F 3 "" H 9400 3250 50  0001 C CNN
+	1    9400 3250
+	1    0    0    -1
+$EndComp
+Wire Wire Line
+	9400 3250 9400 3200
+Wire Wire Line
+	9400 3000 9400 2900
 Wire Wire Line
 	5950 2900 6250 2900
@@
 F 0 "D2" H 4200 3450 50  0000 C CNN
 F 1 "RED_LED" H 4300 3300 50  0000 C CNN
-F 2 "LED_THT:LED_D5.0mm" H 4300 3400 50  0001 C CNN
+F 2 "LED_SMD:LED_0805_2012Metric" H 4300 3400 50  0001 C CNN
 F 3 "~" H 4300 3400 50  0001 C CNN
 	1    4300 3400
@@
 F 0 "D1" H 3900 3450 50  0000 C CNN
 F 1 "GREEN_LED" H 3950 3300 50  0000 C CNN
-F 2 "LED_THT:LED_D5.0mm" H 4000 3400 50  0001 C CNN
+F 2 "LED_SMD:LED_0805_2012Metric" H 4000 3400 50  0001 C CNN
 F 3 "~" H 4000 3400 50  0001 C CNN
 	1    4000 3400
@@
 F 0 "BT1" H 6368 3546 50  0000 L CNN
 F 1 "Battery_Cell" H 6368 3455 50  0000 L CNN
-F 2 "power_supplies:Keystone_18650_Battery_Clip" V 6250 3510 50  0001 C CNN
+F 2 "Connector_JST:JST_PH_B2B-PH-K_1x02_P2.00mm_Vertical" V 6250 3510 50  0001 C CNN
 F 3 "http://www.farnell.com/datasheets/1898890.pdf" V 6250 3510 50  0001 C CNN
 F 4 "https://au.element14.com/keystone/54/battery-clip-18mm-cell-pcb-through/dp/1888422" H 6250 3450 50  0001 C CNN "Supplier"
@@
 Wire Wire Line
 	6900 2900 6900 3000
+$Comp
+L Regulator_Linear:AMS1117 U4
+U 1 1 5C8E6BA3
+P 8750 2900
+F 0 "U4" H 8750 3142 50  0000 C CNN
+F 1 "AMS1117" H 8750 3051 50  0000 C CNN
+F 2 "Package_TO_SOT_SMD:SOT-223-3_TabPin2" H 8750 3100 50  0001 C CNN
+F 3 "http://www.advanced-monolithic.com/pdf/ds1117.pdf" H 8850 2650 50  0001 C CNN
+	1    8750 2900
+	1    0    0    -1
+$EndComp
+Wire Wire Line
+	7950 2900 8450 2900
+Wire Wire Line
+	9050 2900 9100 2900
+Connection ~ 9100 2900
+Wire Wire Line
+	9100 2900 9400 2900
+Connection ~ 9400 2900
+Wire Wire Line
+	9400 2900 9700 2900
 $EndSCHEMATC

Commit message: PCB finished
Parts:
- removed H1, H2, H3, H4: MountingHole, MountingHole:MountingHole_3.2mm_M3_ISO7380, symbol Mechanical:MountingHole
- added Q1: IRF7404, Package_SO:SOIC-8_3.9x4.9mm_P1.27mm, symbol Transistor_FET:IRF7404
- added R14: 10k, Resistor_SMD:R_0805_2012Metric, symbol Device:R_Small
- added SW3: SW_SPST, Button_Switch_THT:SW_CuK_JS202011CQN_DPDT_Straight, symbol Switch:SW_SPST
Connections:
- net labels added: P5_0, P5_1, P_Batt_0, P_Batt_1
- wire segments 58 -> 65
Other:
- moved on the sheet: C10, C11, C9, R10, R11, U4

Commit message: update
Parts:
- removed D1: GREEN_LED, LED_SMD:LED_0805_2012Metric, symbol Device:LED
- removed D2: RED_LED, LED_SMD:LED_0805_2012Metric, symbol Device:LED
- renumbered C11 to C10, C10 to C11, J4 to J1, R14 to R10, R10 to R11, R11 to R14
Connections:
- net labels added: power_status
- wire segments 65 -> 67
Changed lines of the file:
@@
 EESchema Schematic File Version 4
 LIBS:esp32_rs232_adapter-cache
-EELAYER 26 0
+EELAYER 29 0
 EELAYER END
 $Descr A4 11693 8268
@@
 $EndDescr
 $Comp
-L power:GND #PWR018
+L power:GND #PWR01
 U 1 1 5BF53907
 P 2700 3650
-F 0 "#PWR018" H 2700 3400 50  0001 C CNN
+F 0 "#PWR?" H 2700 3400 50  0001 C CNN
 F 1 "GND" H 2705 3477 50  0000 C CNN
 F 2 "" H 2700 3650 50  0001 C CNN
@@
 	8750 2900 8750 3050
 $Comp
-L power:GND #PWR027
+L power:GND #PWR025
 U 1 1 5C832AA9
 P 9600 3250
-F 0 "#PWR027" H 9600 3000 50  0001 C CNN
+F 0 "#PWR?" H 9600 3000 50  0001 C CNN
 F 1 "GND" H 9605 3077 50  0000 C CNN
 F 2 "" H 9600 3250 50  0001 C CNN
@@
 $EndComp
 $Comp
-L power:GND #PWR025
+L power:GND #PWR024
 U 1 1 5C832B16
 P 9250 3250
-F 0 "#PWR025" H 9250 3000 50  0001 C CNN
+F 0 "#PWR?" H 9250 3000 50  0001 C CNN
 F 1 "GND" H 9255 3077 50  0000 C CNN
 F 2 "" H 9250 3250 50  0001 C CNN
@@
 $EndComp
 $Comp
-L power:GND #PWR024
+L power:GND #PWR023
 U 1 1 5C832B83
 P 8750 3350
-F 0 "#PWR024" H 8750 3100 50  0001 C CNN
+F 0 "#PWR?" H 8750 3100 50  0001 C CNN
 F 1 "GND" H 8755 3177 50  0000 C CNN
 F 2 "" H 8750 3350 50  0001 C CNN
@@
 U 1 1 5C841C27
 P 8750 3150
-F 0 "C9" H 8842 3196 50  0000 L CNN
+F 0 "C?" H 8842 3196 50  0000 L CNN
 F 1 "1u" H 8842 3105 50  0000 L CNN
 F 2 "Capacitor_SMD:C_0805_2012Metric" H 8750 3150 50  0001 C CNN
@@
 $EndComp
 $Comp
-L Device:C_Small C11
+L Device:C_Small C10
 U 1 1 5C841CF1
 P 9600 3100
-F 0 "C11" H 9692 3146 50  0000 L CNN
+F 0 "C?" H 9692 3146 50  0000 L CNN
 F 1 "1u" H 9692 3055 50  0000 L CNN
 F 2 "Capacitor_SMD:C_0805_2012Metric" H 9600 3100 50  0001 C CNN
@@
 $EndComp
 $Comp
-L Connector:USB_B_Micro J4
+L Connector:USB_B_Micro J1
 U 1 1 5C4ADCCF
 P 2700 3150
-F 0 "J4" H 2755 3617 50  0000 C CNN
+F 0 "J?" H 2755 3617 50  0000 C CNN
 F 1 "USB_B_Micro" H 2755 3526 50  0000 C CNN
 F 2 "power_supplies:USB_Micro-B_Molex-105017-0001" H 2850 3100 50  0001 C CNN
@@
 	2600 3600 2700 3600
 $Comp
-L Device:C_Small C10
+L Device:C_Small C11
 U 1 1 5C4A11C5
 P 9900 3100
-F 0 "C10" H 9992 3146 50  0000 L CNN
+F 0 "C?" H 9992 3146 50  0000 L CNN
 F 1 "10n" H 9992 3055 50  0000 L CNN
 F 2 "Capacitor_SMD:C_0805_2012Metric" H 9900 3100 50  0001 C CNN
@@
 U 1 1 5C4A145F
 P 9900 3250
-F 0 "#PWR026" H 9900 3000 50  0001 C CNN
+F 0 "#PWR?" H 9900 3000 50  0001 C CNN
 F 1 "GND" H 9905 3077 50  0000 C CNN
 F 2 "" H 9900 3250 50  0001 C CNN
@@
 U 1 1 5C494BB4
 P 6250 3050
-F 0 "F1" H 6250 3235 50  0000 C CNN
+F 0 "F?" H 6250 3235 50  0000 C CNN
 F 1 "4A" H 6250 3144 50  0000 C CNN
 F 2 "Fuse:Fuse_1206_3216Metric" H 6250 3050 50  0001 C CNN
@@
 U 1 1 5C47EED8
 P 3250 2950
-F 0 "R6" H 3309 2996 50  0000 L CNN
+F 0 "R?" H 3309 2996 50  0000 L CNN
 F 1 "0.2" H 3309 2905 50  0000 L CNN
 F 2 "Resistor_SMD:R_0805_2012Metric" H 3250 2950 50  0001 C CNN
@@
 $EndComp
 Wire Wire Line
-	4000 3200 4000 3250
-Wire Wire Line
-	4300 3200 4300 3250
-Wire Wire Line
 	4300 2950 4700 2950
 Connection ~ 4300 2950
@@
 	5900 4000 5900 3950
 $Comp
-L power:GND #PWR021
+L power:GND #PWR018
 U 1 1 5C527D0F
 P 5900 4000
-F 0 "#PWR021" H 5900 3750 50  0001 C CNN
+F 0 "#PWR?" H 5900 3750 50  0001 C CNN
 F 1 "GND" H 5905 3827 50  0000 C CNN
 F 2 "" H 5900 4000 50  0001 C CNN
@@
 	4000 3700 5000 3700
 Wire Wire Line
-	4000 3550 4000 3700
-Wire Wire Line
 	4300 3600 5000 3600
 Wire Wire Line
-	4300 3550 4300 3600
-Wire Wire Line
 	4700 3300 5000 3300
 Wire Wire Line
 	3500 3300 3500 3350
 $Comp
-L power:GND #PWR019
+L power:GND #PWR02
 U 1 1 5C4E7ECD
 P 3500 3350
-F 0 "#PWR019" H 3500 3100 50  0001 C CNN
+F 0 "#PWR?" H 3500 3100 50  0001 C CNN
 F 1 "GND" H 3505 3177 50  0000 C CNN
 F 2 "" H 3500 3350 50  0001 C CNN
@@
 	5400 4000 5400 3950
 $Comp
-L power:GND #PWR020
+L power:GND #PWR017
 U 1 1 5C4BD85A
 P 5400 4000
-F 0 "#PWR020" H 5400 3750 50  0001 C CNN
+F 0 "#PWR?" H 5400 3750 50  0001 C CNN
 F 1 "GND" H 5405 3827 50  0000 C CNN
 F 2 "" H 5400 4000 50  0001 C CNN
@@
 	1    0    0    -1
 $EndComp
-$Comp
-L Device:LED D2
-U 1 1 5C4BD357
-P 4300 3400
-F 0 "D2" H 4200 3450 50  0000 C CNN
-F 1 "RED_LED" H 4300 3300 50  0000 C CNN
-F 2 "LED_SMD:LED_0805_2012Metric" H 4300 3400 50  0001 C CNN
-F 3 "~" H 4300 3400 50  0001 C CNN
-	1    4300 3400
-	0    1    -1   0
-$EndComp
-$Comp
-L Device:LED D1
-U 1 1 5C4BD251
-P 4000 3400
-F 0 "D1" H 3900 3450 50  0000 C CNN
-F 1 "GREEN_LED" H 3950 3300 50  0000 C CNN
-F 2 "LED_SMD:LED_0805_2012Metric" H 4000 3400 50  0001 C CNN
-F 3 "~" H 4000 3400 50  0001 C CNN
-	1    4000 3400
-	0    1    -1   0
-$EndComp
 Wire Wire Line
 	5800 3600 5950 3600
@@
 U 1 1 5C4ADFEE
 P 5950 3400
-F 0 "C8" H 6042 3446 50  0000 L CNN
+F 0 "C?" H 6042 3446 50  0000 L CNN
 F 1 "10u" H 6042 3355 50  0000 L CNN
 F 2 "Capacitor_SMD:C_0805_2012Metric" H 5950 3400 50  0001 C CNN
@@
 U 1 1 5C4AD987
 P 3500 3200
-F 0 "C7" H 3592 3246 50  0000 L CNN
+F 0 "C?" H 3592 3246 50  0000 L CNN
 F 1 "10u" H 3592 3155 50  0000 L CNN
 F 2 "Capacitor_SMD:C_0805_2012Metric" H 3500 3200 50  0001 C CNN
@@
 U 1 1 5C4AD354
 P 4300 3100
-F 0 "R8" H 4359 3146 50  0000 L CNN
+F 0 "R?" H 4359 3146 50  0000 L CNN
 F 1 "200" H 4359 3055 50  0000 L CNN
 F 2 "Resistor_SMD:R_0805_2012Metric" H 4300 3100 50  0001 C CNN
@@
 U 1 1 5C4AD1A5
 P 4000 3100
-F 0 "R7" H 4059 3146 50  0000 L CNN
+F 0 "R?" H 4059 3146 50  0000 L CNN
 F 1 "200" H 4059 3055 50  0000 L CNN
 F 2 "Resistor_SMD:R_0805_2012Metric" H 4000 3100 50  0001 C CNN
@@
 U 1 1 5C4AD007
 P 5900 3850
-F 0 "R9" H 5959 3896 50  0000 L CNN
+F 0 "R?" H 5959 3896 50  0000 L CNN
 F 1 "1.2k" H 5959 3805 50  0000 L CNN
 F 2 "Resistor_SMD:R_0805_2012Metric" H 5900 3850 50  0001 C CNN
@@
 U 1 1 5C495639
 P 5500 3200
-F 0 "U3" H 5400 3515 50  0000 C CNN
+F 0 "U?" H 5400 3515 50  0000 C CNN
 F 1 "TP4056" H 5400 3424 50  0000 C CNN
 F 2 "Package_SO:SSOP-8_3.9x5.05mm_P1.27mm" H 5400 3450 50  0001 C CNN
@@
 U 1 1 5BF52D03
 P 6250 3450
-F 0 "BT1" H 6368 3546 50  0000 L CNN
+F 0 "BT?" H 6368 3546 50  0000 L CNN
 F 1 "Battery_Cell" H 6368 3455 50  0000 L CNN
 F 2 "Connector_JST:JST_PH_B2B-PH-K_1x02_P2.00mm_Vertical" V 6250 3510 50  0001 C CNN
@@
 $EndComp
 $Comp
-L power:+BATT #PWR022
+L power:+BATT #PWR019
 U 1 1 5BF5800F
 P 6250 2850
-F 0 "#PWR022" H 6250 2700 50  0001 C CNN
+F 0 "#PWR?" H 6250 2700 50  0001 C CNN
 F 1 "+BATT" H 6265 3023 50  0000 C CNN
 F 2 "" H 6250 2850 50  0001 C CNN
@@
 $EndComp
 $Comp
-L power:GND #PWR023
+L power:GND #PWR020
 U 1 1 5BF3D77E
 P 6250 3800
-F 0 "#PWR023" H 6250 3550 50  0001 C CNN
+F 0 "#PWR?" H 6250 3550 50  0001 C CNN
 F 1 "GND" H 6255 3627 50  0000 C CNN
 F 2 "" H 6250 3800 50  0001 C CNN
@@
 Vbatt_sig
 $Comp
-L Device:R_Small R10
+L Device:R_Small R11
 U 1 1 5C535CAB
 P 8000 3100
-F 0 "R10" H 8059 3146 50  0000 L CNN
+F 0 "R?" H 8059 3146 50  0000 L CNN
 F 1 "10k" H 8059 3055 50  0000 L CNN
 F 2 "Resistor_SMD:R_0805_2012Metric" H 8000 3100 50  0001 C CNN
@@
 $EndComp
 $Comp
-L Device:R_Small R11
+L Device:R_Small R14
 U 1 1 5C535DD9
 P 8000 3400
-F 0 "R11" H 8059 3446 50  0000 L CNN
+F 0 "R?" H 8059 3446 50  0000 L CNN
 F 1 "10k" H 8059 3355 50  0000 L CNN
 F 2 "Resistor_SMD:R_0805_2012Metric" H 8000 3400 50  0001 C CNN
@@
 U 1 1 5C8E6BA3
 P 9250 2900
-F 0 "U4" H 9250 3142 50  0000 C CNN
+F 0 "U?" H 9250 3142 50  0000 C CNN
 F 1 "AMS1117" H 9250 3051 50  0000 C CNN
 F 2 "Package_TO_SOT_SMD:SOT-223-3_TabPin2" H 9250 3100 50  0001 C CNN
@@
 U 1 1 5C986A9A
 P 7250 3000
-F 0 "Q1" V 7593 3000 50  0000 C CNN
+F 0 "Q?" V 7593 3000 50  0000 C CNN
 F 1 "IRF7404" V 7502 3000 50  0000 C CNN
 F 2 "Package_SO:SOIC-8_3.9x4.9mm_P1.27mm" H 7450 2925 50  0001 L CIN
@@
 Connection ~ 8750 2900
 $Comp
-L power:GND #PWR017
+L power:GND #PWR021
 U 1 1 5C98B42F
 P 7250 3750
-F 0 "#PWR017" H 7250 3500 50  0001 C CNN
+F 0 "#PWR?" H 7250 3500 50  0001 C CNN
 F 1 "GND" H 7255 3577 50  0000 C CNN
 F 2 "" H 7250 3750 50  0001 C CNN
@@
 U 1 1 5C98B4C2
 P 7250 3500
-F 0 "SW3" V 7204 3598 50  0000 L CNN
+F 0 "SW?" V 7204 3598 50  0000 L CNN
 F 1 "SW_SPST" V 7295 3598 50  0000 L CNN
 F 2 "Button_Switch_THT:SW_CuK_JS202011CQN_DPDT_Straight" H 7250 3500 50  0001 C CNN
@@
 	7250 3300 7250 3250
 $Comp
-L Device:R_Small R14
+L Device:R_Small R10
 U 1 1 5C98D447
 P 6850 3100
-F 0 "R14" H 6909 3146 50  0000 L CNN
+F 0 "R?" H 6909 3146 50  0000 L CNN
 F 1 "10k" H 6909 3055 50  0000 L CNN
 F 2 "Resistor_SMD:R_0805_2012Metric" H 6850 3100 50  0001 C CNN
@@
 	8000 2900 8750 2900
 $Comp
-L power:GND #PWR028
+L power:GND #PWR022
 U 1 1 5C9956ED
 P 8000 3600
-F 0 "#PWR028" H 8000 3350 50  0001 C CNN
+F 0 "#PWR?" H 8000 3350 50  0001 C CNN
 F 1 "GND" H 8005 3427 50  0000 C CNN
 F 2 "" H 8000 3600 50  0001 C CNN
@@
 Text Label 6250 3200 0    50   ~ 0
 P_Batt_0
+Wire Wire Line
+	4000 3200 4000 3700
+Wire Wire Line
+	4300 3200 4300 3600
+Text Label 4400 3700 0    50   ~ 0
+power_status
+Text HLabel 4050 3950 2    50   Input ~ 0
+power_status
+Text HLabel 4400 3850 2    50   Input ~ 0
+charge_status
+Wire Wire Line
+	4300 3600 4300 3850
+Wire Wire Line
+	4300 3850 4400 3850
+Connection ~ 4300 3600
+Wire Wire Line
+	4000 3950 4050 3950
+Wire Wire Line
+	4000 3700 4000 3950
+Connection ~ 4000 3700
 $EndSCHEMATC
