File: PCB/power_supply.sch (KiCad schematic (older format))
At the start: 19 parts, among them J1 USB_B_Micro, Q1 IRF7404, SW3 SW_SPST, U3 TP4056, U4 AMS1117

Commit message: work in progress with stuff for cb testing
Changed lines of the file:
@@
 EESchema Schematic File Version 4
 LIBS:esp32_rs232_adapter-cache
-EELAYER 29 0
+EELAYER 26 0
 EELAYER END
 $Descr A4 11693 8268
@@
 $EndDescr
 $Comp
-L power:GND #PWR01
+L power:GND #PWR0103
 U 1 1 5BF53907
 P 2700 3650
-F 0 "#PWR?" H 2700 3400 50  0001 C CNN
+F 0 "#PWR0103" H 2700 3400 50  0001 C CNN
 F 1 "GND" H 2705 3477 50  0000 C CNN
 F 2 "" H 2700 3650 50  0001 C CNN
@@
 	8750 2900 8750 3050
 $Comp
-L power:GND #PWR025
+L power:GND #PWR0104
 U 1 1 5C832AA9
 P 9600 3250
-F 0 "#PWR?" H 9600 3000 50  0001 C CNN
+F 0 "#PWR0104" H 9600 3000 50  0001 C CNN
 F 1 "GND" H 9605 3077 50  0000 C CNN
 F 2 "" H 9600 3250 50  0001 C CNN
@@
 $EndComp
 $Comp
-L power:GND #PWR024
+L power:GND #PWR0105
 U 1 1 5C832B16
 P 9250 3250
-F 0 "#PWR?" H 9250 3000 50  0001 C CNN
+F 0 "#PWR0105" H 9250 3000 50  0001 C CNN
 F 1 "GND" H 9255 3077 50  0000 C CNN
 F 2 "" H 9250 3250 50  0001 C CNN
@@
 $EndComp
 $Comp
-L power:GND #PWR023
+L power:GND #PWR0106
 U 1 1 5C832B83
 P 8750 3350
-F 0 "#PWR?" H 8750 3100 50  0001 C CNN
+F 0 "#PWR0106" H 8750 3100 50  0001 C CNN
 F 1 "GND" H 8755 3177 50  0000 C CNN
 F 2 "" H 8750 3350 50  0001 C CNN
@@
 U 1 1 5C841C27
 P 8750 3150
-F 0 "C?" H 8842 3196 50  0000 L CNN
+F 0 "C9" H 8842 3196 50  0000 L CNN
 F 1 "1u" H 8842 3105 50  0000 L CNN
 F 2 "Capacitor_SMD:C_0805_2012Metric" H 8750 3150 50  0001 C CNN
@@
 U 1 1 5C841CF1
 P 9600 3100
-F 0 "C?" H 9692 3146 50  0000 L CNN
+F 0 "C10" H 9692 3146 50  0000 L CNN
 F 1 "1u" H 9692 3055 50  0000 L CNN
 F 2 "Capacitor_SMD:C_0805_2012Metric" H 9600 3100 50  0001 C CNN
@@
 U 1 1 5C4ADCCF
 P 2700 3150
-F 0 "J?" H 2755 3617 50  0000 C CNN
+F 0 "J1" H 2755 3617 50  0000 C CNN
 F 1 "USB_B_Micro" H 2755 3526 50  0000 C CNN
 F 2 "power_supplies:USB_Micro-B_Molex-105017-0001" H 2850 3100 50  0001 C CNN
@@
 U 1 1 5C4A11C5
 P 9900 3100
-F 0 "C?" H 9992 3146 50  0000 L CNN
+F 0 "C11" H 9992 3146 50  0000 L CNN
 F 1 "10n" H 9992 3055 50  0000 L CNN
 F 2 "Capacitor_SMD:C_0805_2012Metric" H 9900 3100 50  0001 C CNN
@@
 $EndComp
 $Comp
-L power:GND #PWR026
+L power:GND #PWR0107
 U 1 1 5C4A145F
 P 9900 3250
-F 0 "#PWR?" H 9900 3000 50  0001 C CNN
+F 0 "#PWR0107" H 9900 3000 50  0001 C CNN
 F 1 "GND" H 9905 3077 50  0000 C CNN
 F 2 "" H 9900 3250 50  0001 C CNN
@@
 U 1 1 5C494BB4
 P 6250 3050
-F 0 "F?" H 6250 3235 50  0000 C CNN
+F 0 "F1" H 6250 3235 50  0000 C CNN
 F 1 "4A" H 6250 3144 50  0000 C CNN
 F 2 "Fuse:Fuse_1206_3216Metric" H 6250 3050 50  0001 C CNN
@@
 U 1 1 5C47EED8
 P 3250 2950
-F 0 "R?" H 3309 2996 50  0000 L CNN
+F 0 "R6" H 3309 2996 50  0000 L CNN
 F 1 "0.2" H 3309 2905 50  0000 L CNN
 F 2 "Resistor_SMD:R_0805_2012Metric" H 3250 2950 50  0001 C CNN
@@
 	5900 4000 5900 3950
 $Comp
-L power:GND #PWR018
+L power:GND #PWR0108
 U 1 1 5C527D0F
 P 5900 4000
-F 0 "#PWR?" H 5900 3750 50  0001 C CNN
+F 0 "#PWR0108" H 5900 3750 50  0001 C CNN
 F 1 "GND" H 5905 3827 50  0000 C CNN
 F 2 "" H 5900 4000 50  0001 C CNN
@@
 	3500 3300 3500 3350
 $Comp
-L power:GND #PWR02
+L power:GND #PWR0109
 U 1 1 5C4E7ECD
 P 3500 3350
-F 0 "#PWR?" H 3500 3100 50  0001 C CNN
+F 0 "#PWR0109" H 3500 3100 50  0001 C CNN
 F 1 "GND" H 3505 3177 50  0000 C CNN
 F 2 "" H 3500 3350 50  0001 C CNN
@@
 	5400 4000 5400 3950
 $Comp
-L power:GND #PWR017
+L power:GND #PWR0110
 U 1 1 5C4BD85A
 P 5400 4000
-F 0 "#PWR?" H 5400 3750 50  0001 C CNN
+F 0 "#PWR0110" H 5400 3750 50  0001 C CNN
 F 1 "GND" H 5405 3827 50  0000 C CNN
 F 2 "" H 5400 4000 50  0001 C CNN
@@
 U 1 1 5C4ADFEE
 P 5950 3400
-F 0 "C?" H 6042 3446 50  0000 L CNN
+F 0 "C8" H 6042 3446 50  0000 L CNN
 F 1 "10u" H 6042 3355 50  0000 L CNN
 F 2 "Capacitor_SMD:C_0805_2012Metric" H 5950 3400 50  0001 C CNN
@@
 U 1 1 5C4AD987
 P 3500 3200
-F 0 "C?" H 3592 3246 50  0000 L CNN
+F 0 "C7" H 3592 3246 50  0000 L CNN
 F 1 "10u" H 3592 3155 50  0000 L CNN
 F 2 "Capacitor_SMD:C_0805_2012Metric" H 3500 3200 50  0001 C CNN
@@
 U 1 1 5C4AD354
 P 4300 3100
-F 0 "R?" H 4359 3146 50  0000 L CNN
+F 0 "R8" H 4359 3146 50  0000 L CNN
 F 1 "200" H 4359 3055 50  0000 L CNN
 F 2 "Resistor_SMD:R_0805_2012Metric" H 4300 3100 50  0001 C CNN
@@
 U 1 1 5C4AD1A5
 P 4000 3100
-F 0 "R?" H 4059 3146 50  0000 L CNN
+F 0 "R7" H 4059 3146 50  0000 L CNN
 F 1 "200" H 4059 3055 50  0000 L CNN
 F 2 "Resistor_SMD:R_0805_2012Metric" H 4000 3100 50  0001 C CNN
@@
 U 1 1 5C4AD007
 P 5900 3850
-F 0 "R?" H 5959 3896 50  0000 L CNN
+F 0 "R9" H 5959 3896 50  0000 L CNN
 F 1 "1.2k" H 5959 3805 50  0000 L CNN
 F 2 "Resistor_SMD:R_0805_2012Metric" H 5900 3850 50  0001 C CNN
@@
 U 1 1 5C495639
 P 5500 3200
-F 0 "U?" H 5400 3515 50  0000 C CNN
+F 0 "U3" H 5400 3515 50  0000 C CNN
 F 1 "TP4056" H 5400 3424 50  0000 C CNN
 F 2 "Package_SO:SSOP-8_3.9x5.05mm_P1.27mm" H 5400 3450 50  0001 C CNN
@@
 U 1 1 5BF52D03
 P 6250 3450
-F 0 "BT?" H 6368 3546 50  0000 L CNN
+F 0 "BT1" H 6368 3546 50  0000 L CNN
 F 1 "Battery_Cell" H 6368 3455 50  0000 L CNN
 F 2 "Connector_JST:JST_PH_B2B-PH-K_1x02_P2.00mm_Vertical" V 6250 3510 50  0001 C CNN
@@
 $EndComp
 $Comp
-L power:+BATT #PWR019
+L power:+BATT #PWR0111
 U 1 1 5BF5800F
 P 6250 2850
-F 0 "#PWR?" H 6250 2700 50  0001 C CNN
+F 0 "#PWR0111" H 6250 2700 50  0001 C CNN
 F 1 "+BATT" H 6265 3023 50  0000 C CNN
 F 2 "" H 6250 2850 50  0001 C CNN
@@
 $EndComp
 $Comp
-L power:GND #PWR020
+L power:GND #PWR0112
 U 1 1 5BF3D77E
 P 6250 3800
-F 0 "#PWR?" H 6250 3550 50  0001 C CNN
+F 0 "#PWR0112" H 6250 3550 50  0001 C CNN
 F 1 "GND" H 6255 3627 50  0000 C CNN
 F 2 "" H 6250 3800 50  0001 C CNN
@@
 U 1 1 5C535CAB
 P 8000 3100
-F 0 "R?" H 8059 3146 50  0000 L CNN
+F 0 "R11" H 8059 3146 50  0000 L CNN
 F 1 "10k" H 8059 3055 50  0000 L CNN
 F 2 "Resistor_SMD:R_0805_2012Metric" H 8000 3100 50  0001 C CNN
@@
 U 1 1 5C535DD9
 P 8000 3400
-F 0 "R?" H 8059 3446 50  0000 L CNN
+F 0 "R14" H 8059 3446 50  0000 L CNN
 F 1 "10k" H 8059 3355 50  0000 L CNN
 F 2 "Resistor_SMD:R_0805_2012Metric" H 8000 3400 50  0001 C CNN
@@
 U 1 1 5C8E6BA3
 P 9250 2900
-F 0 "U?" H 9250 3142 50  0000 C CNN
+F 0 "U4" H 9250 3142 50  0000 C CNN
 F 1 "AMS1117" H 9250 3051 50  0000 C CNN
 F 2 "Package_TO_SOT_SMD:SOT-223-3_TabPin2" H 9250 3100 50  0001 C CNN
@@
 U 1 1 5C986A9A
 P 7250 3000
-F 0 "Q?" V 7593 3000 50  0000 C CNN
+F 0 "Q1" V 7593 3000 50  0000 C CNN
 F 1 "IRF7404" V 7502 3000 50  0000 C CNN
 F 2 "Package_SO:SOIC-8_3.9x4.9mm_P1.27mm" H 7450 2925 50  0001 L CIN
@@
 Connection ~ 8750 2900
 $Comp
-L power:GND #PWR021
+L power:GND #PWR0113
 U 1 1 5C98B42F
 P 7250 3750
-F 0 "#PWR?" H 7250 3500 50  0001 C CNN
+F 0 "#PWR0113" H 7250 3500 50  0001 C CNN
 F 1 "GND" H 7255 3577 50  0000 C CNN
 F 2 "" H 7250 3750 50  0001 C CNN
@@
 U 1 1 5C98B4C2
 P 7250 3500
-F 0 "SW?" V 7204 3598 50  0000 L CNN
+F 0 "SW3" V 7204 3598 50  0000 L CNN
 F 1 "SW_SPST" V 7295 3598 50  0000 L CNN
 F 2 "Button_Switch_THT:SW_CuK_JS202011CQN_DPDT_Straight" H 7250 3500 50  0001 C CNN
@@
 U 1 1 5C98D447
 P 6850 3100
-F 0 "R?" H 6909 3146 50  0000 L CNN
+F 0 "R10" H 6909 3146 50  0000 L CNN
 F 1 "10k" H 6909 3055 50  0000 L CNN
 F 2 "Resistor_SMD:R_0805_2012Metric" H 6850 3100 50  0001 C CNN
@@
 	8000 2900 8750 2900
 $Comp
-L power:GND #PWR022
+L power:GND #PWR0114
 U 1 1 5C9956ED
 P 8000 3600
-F 0 "#PWR?" H 8000 3350 50  0001 C CNN
+F 0 "#PWR0114" H 8000 3350 50  0001 C CNN
 F 1 "GND" H 8005 3427 50  0000 C CNN
 F 2 "" H 8000 3600 50  0001 C CNN
